File: pcbs/dreamebreakout-usb_c/kicad/DreameBreakout.kicad_sch (KiCad schematic)
At the start: 10 parts, among them J1 SoC Breakout, J1.1 To Robot SoC, J1.2 To Robot MCU, J2 MCU Breakout, J3 OTG_USB, SW1 SoC_Boot_SEL_BTN

Commit message: Replaced micro-USB with USB-C receptacle. Also added a second Resistor for symeptric pluggablility
Parts:
- added R2: 5.1kΩ±20%, Resistor_THT:R_Axial_DIN0204_L3.6mm_D1.6mm_P7.62mm_Horizontal, symbol PCM_SL_Resistors:Resistor
Connections:
- net SoC_GND: now also R2.2
- net at USB-C1.B5 (CC2): now also R2.1
Changed lines of the file:
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@@
+	(wire
+		(pts
+			(xy 168.91 77.47) (xy 168.91 88.9)
+		)
+		(stroke
+			(width 0)
+			(type default)
+		)
+	)
 	(wire
 		(pts
@@
 		(property "Intersheetrefs" "${INTERSHEET_REFS}"
 			(at 123.9098 75.0094 0)
+			(effects
+				(font
+					(size 1.27 1.27)
+				)
+				(justify left)
+				(hide yes)
+			)
+		)
+	)
+	(global_label "SoC_GND"
+		(shape input)
+		(at 168.91 96.52 0)
+		(fields_autoplaced yes)
+		(effects
+			(font
+				(size 1.27 1.27)
+			)
+			(justify left)
+		)
+		(property "Intersheetrefs" "${INTERSHEET_REFS}"
+			(at 180.3618 96.52 0)
 			(effects
 				(font
@@
 					(unit 1)
 				)
+			)
+		)
+	)
+	(symbol
+		(lib_id "PCM_SL_Resistors:Resistor")
+		(at 168.91 92.71 270)
+		(unit 1)
+		(exclude_from_sim no)
+		(in_bom yes)
+		(on_board yes)
+		(dnp no)
+		(fields_autoplaced yes)
+		(property "Reference" "R2"
+			(at 166.37 93.9801 90)
+			(effects
+				(font
+					(size 1.27 1.27)
+				)
+				(justify right)
+			)
+		)
+		(property "Value" "5.1kΩ±20%"
+			(at 166.37 91.4401 90)
+			(effects
+				(font
+					(size 1.27 1.27)
+				)
+				(justify right)
+			)
+		)
+		(property "Footprint" "Resistor_THT:R_Axial_DIN0204_L3.6mm_D1.6mm_P7.62mm_Horizontal"
+			(at 164.592 93.599 0)
+			(effects
+				(font
+					(size 1.27 1.27)
+				)
+				(hide yes)
+			)
+		)
+		(property "Datasheet" ""
+			(at 168.91 93.218 0)
+			(effects
+				(font
+					(size 1.27 1.27)
+				)
+				(hide yes)
+			)
+		)
+		(property "Description" "1/4W Resistor"
+			(at 168.91 92.71 0)
+			(effects
+				(font
+					(size 1.27 1.27)
+				)
+				(hide yes)
+			)
+		)
+		(pin "1"
+		)
+		(pin "2"
+		)
+		(instances
+			(project "DreameBreakout"
+				(path "/ea31f51c-3f0e-4e37-9fd4-9e1b1b7d7784"
+					(reference "R2")
+					(unit 1)
+				)
